File: Design Files/Exploding Capacitors Lab/poorDuino/V1I1/poorDuino.brd (EAGLE design)
At the start: 68.6 x 53.3 mm, 25 parts, among them IC1 LD117AS33TR, IC2 LD117AS50TR, X1 POWERSUPPLY_DC21MMX, Y2 CSTCE16M0V53-R0 16MHZ

Commit message: PCB layout
Parts:
- added JP1: (no value), pinhead:1X03
- added R5, R6: 4K7, SmartPrj:R0805
- added SJ1, SJ2: (no value), jumper:SJ
- moved C7 92.4 mm to (46.4, 9.78), turned to 180 degrees
- moved 3V3 79.4 mm to (5.33, 26.0), turned to 90 degrees
- moved R4 78.5 mm to (10.2, 26.0), turned to 180 degrees
- moved C3 63.1 mm to (5.33, 29.2), turned to 180 degrees
- moved C2 61.2 mm to (10.2, 29.2), turned to 180 degrees
- moved C5 60.3 mm to (10.2, 15.2), turned to 180 degrees
- moved IC2 52.9 mm to (7.62, 34.3), turned to 270 degrees
- moved C1 46.8 mm to (5.33, 15.2), turned to 180 degrees
- moved IC1 38.1 mm to (7.62, 20.3), turned to 270 degrees
- moved R1 22.1 mm to (6.35, 45.1), turned to 0 degrees
- moved D1 9.77 mm to (17.5, 11.7)
- moved R3 5.78 mm to (10.2, 39.6), turned to 180 degrees
- moved 5V 4.58 mm to (5.33, 39.6), turned to 90 degrees
- moved PC1 4.49 mm to (20.7, 4.57)
- moved C6 0.90 mm to (42.8, 9.78)
Connections:
- new net N$6: R5.1, SJ1.1
- new net N$7: R6.1, SJ2.1
- new net V+: C6.2, ICSP.2, JP1.2, POWER.2, R1.2, R5.2, R6.2, ZU4.20, ZU4.7
- net +3V3: now also JP1.3
- net +5V: now also JP1.1; no longer C6.2, ICSP.2, POWER.2, R1.2, ZU4.20, ZU4.7
- net AD4/SDA: now also SJ2.2
- net AD5/SCL: now also SJ1.2
Routing:
- net V+: track 0.00 -> 128.2 mm, vias 0 -> 3
- net AREF: track 0.00 -> 81.1 mm, vias 0 -> 2
- net VCC: track 0.00 -> 80.4 mm, vias 0 -> 1
- net RESET: track 5.52 -> 85.8 mm, vias 0 -> 1
- net AD5/SCL: track 10.3 -> 89.9 mm, vias 0 -> 2
- net AD4/SDA: track 10.4 -> 89.6 mm
- net +5V: track 0.00 -> 59.8 mm, vias 0 -> 1
- net +3V3: track 0.00 -> 54.2 mm
- net MOSI: track 56.2 -> 91.8 mm, vias 0 -> 1
- net MISO: track 47.1 -> 71.4 mm, vias 0 -> 1
- net PWRIN: track 0.00 -> 15.0 mm
- net N$7: track 0.00 -> 3.73 mm, vias 0 -> 1
- net N$6: track 0.00 -> 3.47 mm, vias 0 -> 1
- net N$3: track 0.00 -> 2.93 mm
- net N$1: track 0.00 -> 2.93 mm
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- added copper zone on layer 1, net GND
- added copper zone on layer 16, net GND
Other:
- board text added: "ANALOG"
- board text removed: "ANALOG IN"

Commit message: PCB layout update
Parts:
- moved R1 1.91 mm to (6.35, 43.2)
- moved 5V 0.38 mm to (5.33, 40.0)
- moved R3 0.38 mm to (10.2, 40.0)
Routing:
- net RESET: track 85.8 -> 156.5 mm, vias 1 -> 4
- net AREF: track 81.1 -> 83.0 mm
- net AD5/SCL: track 89.9 -> 90.9 mm
- net GND: vias 21 -> 27

Commit message: PCB layout
Parts:
- moved PC1 0.64 mm to (20.1, 4.57)
Routing:
- net MOSI: track 91.8 -> 96.4 mm
- net AD4/SDA: track 89.6 -> 92.5 mm
- net AREF: track 83.0 -> 80.7 mm
- net V+: track 128.1 -> 126.4 mm
- net N$2: track 0.00 -> 1.15 mm
- net AD5/SCL: track 90.9 -> 89.9 mm
- net N$4: track 0.00 -> 0.93 mm
- net RESET: track 156.5 -> 157.4 mm
- net SS: track 49.7 -> 50.3 mm

Commit message: PCB update
Routing:
- net RESET: track 157.4 -> 158.5 mm
- net SS: track 50.3 -> 51.3 mm
- net MOSI: track 96.4 -> 97.5 mm
- net +3V3: track 54.6 -> 53.6 mm
- net +5V: track 59.8 -> 59.3 mm
